Commit message: new and improve

File: gp8_simulation/urdf/gp8_macro_gazebo.xacro (robot description, xacro)
@@ -4,4 +4,10 @@
     <xacro:include filename="$(find gp8_simulation)/urdf/gazebo_gp8_plugin.xacro" />
     	<xacro:transmitions prefix=""/>
+    <xacro:macro name="material_yaskawa_blue">
+    <material name="">
+      <color rgba="${color_yaskawa_blue}"/>
+    </material>
+  </xacro:macro>
+    <xacro:property name="color_yaskawa_blue" value="${33/255} ${38/255} ${191/255} 1.0"/>
     <!-- Properties -->
     <!-- <material name="yaskawa_blue">
@@ -18,5 +24,5 @@
                 <mesh filename="package://motoman_gp8_support/meshes/visual/gp8_base_link.stl"/>
             </geometry>
-            <material name="yaskawa_blue"/>
+            <xacro:material_yaskawa_blue/>
         </visual>
         <collision>
@@ -35,5 +41,5 @@
                 <mesh filename="package://motoman_gp8_support/meshes/visual/gp8_link_1_s.stl"/>
             </geometry>
-            <material name="yaskawa_blue"/>
+            <xacro:material_yaskawa_blue/>
         </visual>
         <collision>
@@ -52,5 +58,5 @@
                 <mesh filename="package://motoman_gp8_support/meshes/visual/gp8_link_2_l.stl"/>
             </geometry>
-            <material name="yaskawa_blue"/>
+            <xacro:material_yaskawa_blue/>
         </visual>
         <collision>
@@ -69,5 +75,5 @@
                 <mesh filename="package://motoman_gp8_support/meshes/visual/gp8_link_3_u.stl"/>
             </geometry>
-            <material name="yaskawa_blue"/>
+            <xacro:material_yaskawa_blue/>
         </visual>
         <collision>
@@ -86,5 +92,5 @@
                 <mesh filename="package://motoman_gp8_support/meshes/visual/gp8_link_4_r.stl"/>
             </geometry>
-            <material name="yaskawa_blue"/>
+            <xacro:material_yaskawa_blue/>
         </visual>
         <collision>
@@ -103,5 +109,5 @@
                 <mesh filename="package://motoman_gp8_support/meshes/visual/gp8_link_5_b.stl"/>
             </geometry>
-            <material name="yaskawa_blue"/>
+            <xacro:material_yaskawa_blue/>
         </visual>
         <collision>
@@ -120,5 +126,5 @@
                 <mesh filename="package://motoman_gp8_support/meshes/visual/gp8_link_6_t.stl"/>
             </geometry>
-            <material name="yaskawa_blue"/>
+            <xacro:material_yaskawa_blue/>
         </visual>
         <collision>
